Commit message: created new model, continued cleaning and labeling for code

File: models/raw/bodyv7.urdf (robot description, URDF)
Before this commit: robot arm, 3 links, 2 joints
Links:
- removed link torso
- added link base_link, mass 5.3999999999999995; collision box size=0.03 0.05 0.025; visual box size=0.03 0.05 0.025
- added link head, mass 10.799999999999999; collision box size=0.03 0.05 0.05; visual box size=0.03 0.05 0.05
- added link left_calf, mass 1.875; collision box size=0.022 0.022 0.1; visual box size=0.022 0.022 0.1
- added link left_delt, mass 1.5; collision box size=0.03 0.03 0.03; visual box size=0.03 0.03 0.03
- added link left_foot, mass 0.1875; collision box size=0.045 0.022 0.01; visual box size=0.045 0.022 0.01
- added link left_lower_arm, mass 1.0875; collision box size=0.022 0.022 0.065; visual box size=0.022 0.022 0.065
- added link left_upper_arm, mass 1.0875; collision box size=0.022 0.022 0.065; visual box size=0.022 0.022 0.065
- added link low_torso, mass 13.95; collision box size=0.03 0.05 0.065; visual box size=0.03 0.05 0.065
- added link right_calf, mass 1.875; collision box size=0.022 0.022 0.1; visual box size=0.022 0.022 0.1
- added link right_delt, mass 1.5; collision box size=0.03 0.03 0.03; visual box size=0.03 0.03 0.03
- added link right_foot, mass 0.1875; collision box size=0.045 0.022 0.01; visual box size=0.045 0.022 0.01
- added link right_lower_arm, mass 1.0875; collision box size=0.022 0.022 0.065; visual box size=0.022 0.022 0.065
- added link right_upper_arm, mass 1.0875; collision box size=0.022 0.022 0.065; visual box size=0.022 0.022 0.065
- added link upper_torso, mass 13.95; collision box size=0.03 0.05 0.065; visual box size=0.03 0.05 0.065
- link left_thigh: mass None -> 1.875; geometry collision box size=0.022 0.022 0.1; visual box size=0.022 0.022 0.1
- link right_thigh: mass None -> 1.875; geometry collision box size=0.022 0.022 0.1; visual box size=0.022 0.022 0.1
Joints:
- removed joint left_hip_flexor
- removed joint right_hip_flexor
- added joint bend_low_torso: type revolute, parent base_link, child low_torso, origin xyz=0 0 0, axis 0 1 0, limit lower=-0.8 upper=0.8 effort=20.0 velocity=20.0
- added joint gaze: type revolute, parent upper_torso, child head, origin xyz=0 0 .058, axis 0 0 1, limit lower=-0.8 upper=0.8 effort=20.0 velocity=20.0
- added joint left_ankle: type revolute, parent left_calf, child left_foot, origin xyz=-.015 0 -.1, axis 0 1 0, limit lower=-0.8 upper=0.8 effort=20.0 velocity=20.0
- added joint left_elbow: type revolute, parent left_upper_arm, child left_lower_arm, origin xyz=.015 0 -.055, axis 0 1 0, limit lower=-1.2 upper=0 effort=20.0 velocity=20.0
- added joint left_hip_joint: type revolute, parent base_link, child left_thigh, origin xyz=0 -.014 0, axis 0 1 0, limit lower=-1.2 upper=1.2 effort=20.0 velocity=20.0
- added joint left_knee: type revolute, parent left_thigh, child left_calf, origin xyz=.02 0 -.09, axis 0 1 0, limit lower=0 upper=1.2 effort=20.0 velocity=20.0
- added joint left_shoulder_x: type revolute, parent upper_torso, child left_delt, origin xyz=0 -.035 .05, axis 1 0 0, limit lower=0 upper=1.5 effort=20.0 velocity=20.0
- added joint left_shoulder_y: type revolute, parent left_delt, child left_upper_arm, origin xyz=0 0 -.015, axis 0 1 0, limit lower=-1.2 upper=1.2 effort=20.0 velocity=20.0
- added joint right_ankle: type revolute, parent right_calf, child right_foot, origin xyz=-.015 0 -.1, axis 0 1 0, limit lower=-0.8 upper=0.8 effort=20.0 velocity=20.0
- added joint right_elbow: type revolute, parent right_upper_arm, child right_lower_arm, origin xyz=.015 0 -.055, axis 0 1 0, limit lower=-1.2 upper=0 effort=20.0 velocity=20.0
- added joint right_hip_joint: type revolute, parent base_link, child right_thigh, origin xyz=0 .014 0, axis 0 1 0, limit lower=-1.2 upper=1.2 effort=20.0 velocity=20.0
- added joint right_knee: type revolute, parent right_thigh, child right_calf, origin xyz=.02 0 -.09, axis 0 1 0, limit lower=0 upper=1.2 effort=20.0 velocity=20.0
- added joint right_shoulder_x: type revolute, parent upper_torso, child right_delt, origin xyz=0 .035 .05, axis 1 0 0, limit lower=0 upper=1.5 effort=20.0 velocity=20.0
- added joint right_shoulder_y: type revolute, parent right_delt, child right_upper_arm, origin xyz=0 0 -.015, axis 0 1 0, limit lower=-1.2 upper=1.2 effort=20.0 velocity=20.0
- added joint twist_upper_torso: type revolute, parent low_torso, child upper_torso, origin xyz=0 0 .075, axis 0 0 1, limit lower=-0.8 upper=0.8 effort=20.0 velocity=20.0

File: models/xacro/bodyv7.urdf.xacro (robot description, xacro)
@@ -1,9 +1,11 @@
 <?xml version="1.0"?>
-<robot xmlns:xacro="http://www.ros.org/wiki/xacro" name="arm">
-<xacro:property name="total_weight" value="20" /> <!--KG-->
-<xacro:property name="torso_weight" value="${total_weight * 0.5}" />
-<xacro:property name="leg_weight" value="${(total_weight - torso_weight) * 0.25}" />
-<xacro:property name="torso_length" value="2.5"/>
-<xacro:property name="leg_length" value="1.5"/>
+<robot xmlns:xacro="http://www.ros.org/wiki/xacro" name="Robot 7">
+<xacro:property name="total_weight" value="75" /> <!--KG-->
+<xacro:property name="torso_weight" value="${total_weight * 0.6}" />
+<xacro:property name="leg_weight" value="${total_weight * .15}" />
+<xacro:property name="arm_weight" value="${total_weight * .05}" />
+<xacro:property name="pi" value="3.14"/>
+<xacro:property name="Cyan" value="0 1.0 1.0 1.0"/>
+<xacro:property name="Lilac" value=".8 .6 1.0 1.0"/>
 <xacro:macro name="solid_sphere_inertia_tensors" params="mass radius" >
     <inertial>
@@ -26,54 +28,30 @@
     </inertial>
 </xacro:macro>
-<xacro:macro name="cuboid_inertia_tensors" params="weight length" >
+<xacro:macro name="cuboid_inertia_tensors" params="mass length" >
     <inertial>
         <origin xyz="0.0 0.0 0.0" rpy="0.0 0.0 0.0"/>
-        <mass value="${weight}"/>
+        <mass value="${mass}"/>
         <inertia
-        ixx="${(weight/12)*((length*length*.025)+(length*length*0.0225))}" ixy="0.0" ixz="0.0"
-        iyy="${(weight/12)*((length*length)+(length*length*0.0225))}" iyz="0.0"
-        izz="${(weight/12)*((length*length)+(length*length*0.025))}"/>
+        ixx="${(mass/12)*((length*length*.025)+(length*length*0.0225))}" ixy="0.0" ixz="0.0"
+        iyy="${(mass/12)*((length*length)+(length*length*0.0225))}" iyz="0.0"
+        izz="${(mass/12)*((length*length)+(length*length*0.025))}"/>
     </inertial>
 </xacro:macro>
-ixx ixy ixz
-    iyy iyz
-        izz
-<xacro:macro name="joint_ball" params="name offset">
+<xacro:macro name="cuboid" params="name mass x_len y_len z_len origin rpy">
     <link name="${name}">
         <visual>
             <geometry>
-                <sphere radius="0.01"/>
+                <box size="${x_len} ${y_len} ${z_len}"/>
             </geometry>
-            <origin xyz="${offset}"/>
+            <origin xyz="${origin}" rpy="${rpy}"/>
         </visual>
         <collision>
             <geometry>
-                <sphere radius="0.01"/>
+                <box size="${x_len} ${y_len} ${z_len}"/>
             </geometry>
-            <origin xyz="${offset}"/>
+            <origin xyz="${origin}" rpy="${rpy}"/>
         </collision>
+        <xacro:cuboid_inertia_tensors mass="${mass}" length="${z_len}"/>
     </link>
-</xacro:macro>
-<xacro:macro name="limb" params="name length offset rpy">
-    <link name="${name}">
-        <visual>
-            <geometry>
-                <cylinder radius="0.0050" length="${length}"/>
-            </geometry>
-            <origin xyz="${offset}" rpy="${rpy}"/>
-        </visual>
-        <collision>
-            <geometry>
-                <cylinder radius="0.0050" length="${length}"/>
-            </geometry>
-            <origin xyz="${offset}" rpy="${rpy}"/>
-        </collision>
-    </link>
-</xacro:macro>
-<xacro:macro name="affix" params="name parent child">
-    <joint name="${name}" type="fixed">
-        <parent link="${parent}"/>
-        <child link="${child}"/>
-    </joint>
 </xacro:macro>
 <xacro:macro name="revolve" params="name parent child hi lo axis offset">
@@ -86,7 +64,40 @@
     </joint>
 </xacro:macro>
-<xacro:joint_ball name="base_link" offset="0 0 0"/>
-<!-- Limbs-->
-<!-- Fixed Joints-->
-<!-- Revolute Joints-->
+<xacro:cuboid name="base_link" mass="${torso_weight * .12}" x_len=".03" y_len=".05" z_len=".025" origin="0 0 0" rpy="0 0 0"/>
+<!-- Torso Links-->
+<xacro:cuboid name="low_torso" mass="${torso_weight * .31}" x_len=".03" y_len=".05" z_len=".065" origin="0 0 .045" rpy="0 0 0"/>
+<xacro:cuboid name="upper_torso" mass="${torso_weight * .31}" x_len=".03" y_len=".05" z_len=".065" origin="0 0 .0325" rpy="0 0 0"/>
+<xacro:cuboid name="head" mass="${torso_weight * .24}" x_len=".03" y_len=".05" z_len=".05" origin="0 0 .0325" rpy="0 0 0"/>
+<!-- Torso joints-->
+<xacro:revolve name="bend_low_torso" parent="base_link" child="low_torso" hi=".8" lo="-.8" axis="0 1 0" offset="0 0 0"/>
+<xacro:revolve name="twist_upper_torso" parent="low_torso" child="upper_torso" hi=".8" lo="-.8" axis="0 0 1" offset="0 0 .075"/>
+<xacro:revolve name="gaze" parent="upper_torso" child="head" hi=".8" lo="-.8" axis="0 0 1" offset="0 0 .058"/>
+<!-- Arm Links-->
+<xacro:cuboid name="right_delt" mass="${arm_weight * .4}" x_len=".03" y_len=".03" z_len=".03" origin="0 0 0" rpy="0 0 0"/>
+<xacro:cuboid name="right_upper_arm" mass="${arm_weight * .29}" x_len=".022" y_len=".022" z_len=".065" origin=".005 0 -.025" rpy="0 -${pi/15} 0"/>
+<xacro:cuboid name="right_lower_arm" mass="${arm_weight * .29}" x_len=".022" y_len=".022" z_len=".065" origin=".005 0 -.025" rpy="0 -${pi/10} 0"/>
+<xacro:cuboid name="left_delt" mass="${arm_weight * .4}" x_len=".03" y_len=".03" z_len=".03" origin="0 0 0" rpy="0 0 0"/>
+<xacro:cuboid name="left_upper_arm" mass="${arm_weight * .29}" x_len=".022" y_len=".022" z_len=".065" origin=".005 0 -.025" rpy="0 -${pi/15} 0"/>
+<xacro:cuboid name="left_lower_arm" mass="${arm_weight * .29}" x_len=".022" y_len=".022" z_len=".065" origin=".005 0 -.025" rpy="0 -${pi/10} 0"/>
+<!-- Arm joints-->
+<xacro:revolve name="right_shoulder_x" parent="upper_torso" child="right_delt" hi="1.5" lo="0" axis="1 0 0" offset="0 .035 .05"/>
+<xacro:revolve name="right_shoulder_y" parent="right_delt" child="right_upper_arm" hi="1.2" lo="-1.2" axis="0 1 0" offset="0 0 -.015"/>
+<xacro:revolve name="right_elbow" parent="right_upper_arm" child="right_lower_arm" hi="0" lo="-1.2" axis="0 1 0" offset=".015 0 -.055"/>
+<xacro:revolve name="left_shoulder_x" parent="upper_torso" child="left_delt" hi="1.5" lo="0" axis="1 0 0" offset="0 -.035 .05"/>
+<xacro:revolve name="left_shoulder_y" parent="left_delt" child="left_upper_arm" hi="1.2" lo="-1.2" axis="0 1 0" offset="0 0 -.015"/>
+<xacro:revolve name="left_elbow" parent="left_upper_arm" child="left_lower_arm" hi="0" lo="-1.2" axis="0 1 0" offset=".015 0 -.055"/>
+<!-- Leg Links-->
+<xacro:cuboid name="right_thigh" mass="${arm_weight * .5}" x_len=".022" y_len=".022" z_len=".1" origin=".01 0 -.05" rpy="0 -${pi/15} 0"/>
+<xacro:cuboid name="left_thigh" mass="${arm_weight * .5}" x_len=".022" y_len=".022" z_len=".1" origin=".01 0 -.05" rpy="0 -${pi/15} 0"/>
+<xacro:cuboid name="left_calf" mass="${arm_weight * .5}" x_len=".022" y_len=".022" z_len=".1" origin="-.005 0 -.05" rpy="0 ${pi/20} 0"/>
+<xacro:cuboid name="right_calf" mass="${arm_weight * .5}" x_len=".022" y_len=".022" z_len=".1" origin="-.005 0 -.05" rpy="0 ${pi/20} 0"/>
+<xacro:cuboid name="right_foot" mass="${arm_weight * .05}" x_len=".045" y_len=".022" z_len=".01" origin=".015 0 0" rpy="0 0 0"/>
+<xacro:cuboid name="left_foot" mass="${arm_weight * .05}" x_len=".045" y_len=".022" z_len=".01" origin=".015 0 0" rpy="0 0 0"/>
+<!-- Leg joints-->
+<xacro:revolve name="right_hip_joint" parent="base_link" child="right_thigh" hi="1.2" lo="-1.2" axis="0 1 0" offset="0 .014 0"/>
+<xacro:revolve name="left_hip_joint" parent="base_link" child="left_thigh" hi="1.2" lo="-1.2" axis="0 1 0" offset="0 -.014 0"/>
+<xacro:revolve name="right_knee" parent="right_thigh" child="right_calf" hi="1.2" lo="0" axis="0 1 0" offset=".02 0 -.09"/>
+<xacro:revolve name="left_knee" parent="left_thigh" child="left_calf" hi="1.2" lo="0" axis="0 1 0" offset=".02 0 -.09"/>
+<xacro:revolve name="right_ankle" parent="right_calf" child="right_foot" hi=".8" lo="-.8" axis="0 1 0" offset="-.015 0 -.1"/>
+<xacro:revolve name="left_ankle" parent="left_calf" child="left_foot" hi=".8" lo="-.8" axis="0 1 0" offset="-.015 0 -.1"/>
 </robot>

Commit message: Updated Dir structure

File: models/raw/bodyv7.urdf (robot description, URDF)
Before this commit: robot Robot 7, 16 links, 15 joints
Joints:
- joint bend_low_torso: limit lower=-0.8 upper=0.8 effort=20.0 velocity=20.0 -> lower=-0.8 upper=0.8 effort=200.0 velocity=25.0
- joint gaze: limit lower=-0.8 upper=0.8 effort=20.0 velocity=20.0 -> lower=-0.8 upper=0.8 effort=200.0 velocity=25.0
- joint left_ankle: limit lower=-0.8 upper=0.8 effort=20.0 velocity=20.0 -> lower=-0.8 upper=0.8 effort=200.0 velocity=25.0
- joint left_elbow: limit lower=-1.2 upper=0 effort=20.0 velocity=20.0 -> lower=-1.2 upper=0 effort=200.0 velocity=25.0
- joint left_hip_joint: limit lower=-1.2 upper=1.2 effort=20.0 velocity=20.0 -> lower=-1.2 upper=1.2 effort=200.0 velocity=25.0
- joint left_knee: limit lower=0 upper=1.2 effort=20.0 velocity=20.0 -> lower=0 upper=1.2 effort=200.0 velocity=25.0
- joint left_shoulder_x: limit lower=0 upper=1.5 effort=20.0 velocity=20.0 -> lower=-1.5 upper=0 effort=200.0 velocity=25.0
- joint left_shoulder_y: limit lower=-1.2 upper=1.2 effort=20.0 velocity=20.0 -> lower=-1.2 upper=1.2 effort=200.0 velocity=25.0
- joint right_ankle: limit lower=-0.8 upper=0.8 effort=20.0 velocity=20.0 -> lower=-0.8 upper=0.8 effort=200.0 velocity=25.0
- joint right_elbow: limit lower=-1.2 upper=0 effort=20.0 velocity=20.0 -> lower=-1.2 upper=0 effort=200.0 velocity=25.0
- joint right_hip_joint: limit lower=-1.2 upper=1.2 effort=20.0 velocity=20.0 -> lower=-1.2 upper=1.2 effort=200.0 velocity=25.0
- joint right_knee: limit lower=0 upper=1.2 effort=20.0 velocity=20.0 -> lower=0 upper=1.2 effort=200.0 velocity=25.0
- joint right_shoulder_x: limit lower=0 upper=1.5 effort=20.0 velocity=20.0 -> lower=0 upper=1.5 effort=200.0 velocity=25.0
- joint right_shoulder_y: limit lower=-1.2 upper=1.2 effort=20.0 velocity=20.0 -> lower=-1.2 upper=1.2 effort=200.0 velocity=25.0
- joint twist_upper_torso: limit lower=-0.8 upper=0.8 effort=20.0 velocity=20.0 -> lower=-0.8 upper=0.8 effort=200.0 velocity=25.0

File: models/xacro/bodyv7.urdf.xacro (robot description, xacro)
@@ -58,5 +58,5 @@
         <parent link="${parent}"/>
         <child link="${child}"/>
-        <limit lower="${lo}" upper="${hi}" effort="20.0" velocity="20.0"/>
+        <limit lower="${lo}" upper="${hi}" effort="200.0" velocity="25.0"/>
         <origin xyz="${offset}"/>
         <axis xyz="${axis}"/>
@@ -83,5 +83,5 @@
 <xacro:revolve name="right_shoulder_y" parent="right_delt" child="right_upper_arm" hi="1.2" lo="-1.2" axis="0 1 0" offset="0 0 -.015"/>
 <xacro:revolve name="right_elbow" parent="right_upper_arm" child="right_lower_arm" hi="0" lo="-1.2" axis="0 1 0" offset=".015 0 -.055"/>
-<xacro:revolve name="left_shoulder_x" parent="upper_torso" child="left_delt" hi="1.5" lo="0" axis="1 0 0" offset="0 -.035 .05"/>
+<xacro:revolve name="left_shoulder_x" parent="upper_torso" child="left_delt" hi="0" lo="-1.5" axis="1 0 0" offset="0 -.035 .05"/>
 <xacro:revolve name="left_shoulder_y" parent="left_delt" child="left_upper_arm" hi="1.2" lo="-1.2" axis="0 1 0" offset="0 0 -.015"/>
 <xacro:revolve name="left_elbow" parent="left_upper_arm" child="left_lower_arm" hi="0" lo="-1.2" axis="0 1 0" offset=".015 0 -.055"/>
